File: Planty.kicad_sch (KiCad schematic)
At the start: 41 parts, among them J1 USB_C_Receptacle_USB2.0, Q1 WPM2031, U1 ESP32-C3, U2 MCP73831-2-OT, U3 MIC5504-3.3YM5, Y1 Crystal_GND24

Commit message: finished v1.0.0
Parts:
- removed AE1: Antenna_Chip, RF_Antenna:Texas_SWRA117D_2.4GHz_Left, symbol Device:Antenna_Chip
- removed C1, C3: 10p, Capacitor_SMD:C_0402_1005Metric, symbol Device:C
- removed C2, C4: 3p3, Capacitor_SMD:C_0402_1005Metric, symbol Device:C
- removed C5: 10u, Capacitor_SMD:C_0402_1005Metric, symbol Device:C
- removed C6, C7: 100n, Capacitor_SMD:C_0402_1005Metric, symbol Device:C
- removed L1: 2n2, Inductor_SMD:L_0402_1005Metric, symbol Device:L
- removed U1: ESP32-C3, Package_DFN_QFN:QFN-32-1EP_5x5mm_P0.5mm_EP3.45x3.45mm, symbol Espressif:ESP32-C3
- removed Y1: Crystal_GND24, Crystal:Crystal_SMD_2016-4Pin_2.0x1.6mm, symbol Device:Crystal_GND24
- added U1: ESP32-C3-WROOM-02, Espressif:ESP32-C3-WROOM-02, symbol Espressif:ESP32-C3-WROOM-02
- BT1: footprint Connector_Molex:Molex_PicoBlade_53261-0271_1x02-1MP_P1.25mm_Horizontal -> Connector_JST:JST_PH_S2B-PH-SM4-TB_1x02-1MP_P2.00mm_Horizontal
- C10, C11, C12, C13, C8, C9: footprint Capacitor_SMD:C_0402_1005Metric -> Capacitor_SMD:C_0805_2012Metric
- D1, D3: footprint LED_SMD:LED_0402_1005Metric -> LED_SMD:LED_0805_2012Metric
- R1, R10, R11, R12, R13, R14, R2, R3, R5, R6, R7, R8, R9: footprint Resistor_SMD:R_0402_1005Metric -> Resistor_SMD:R_0805_2012Metric
- R4: value 3k -> 10k; footprint Resistor_SMD:R_0402_1005Metric -> Resistor_SMD:R_0805_2012Metric
Connections:
- net +3V3: now also R6.1, R7.1, U1.1 (3V3); no longer R6.2, R7.2
- net ADC: now also U1.3 (GPIO4/ADC1_CH4)
- net ADC_EN: now also U1.15 (GPIO3/ADC1_CH3)
- net D+: now also U1.14 (GPIO19/USB_D+)
- net D-: now also U1.13 (GPIO18/USB_D-)
- net GND: now also J1.S1 (SHIELD), U1.19 (GND), U1.9 (GND)
- net OUT: now also U1.18 (GPIO0/ADC1_CH0/XTAL_32K_P)
- net PULSE: now also U1.17 (GPIO1/ADC1_CH1/XTAL_32K_N)
- net at R3.2: now also U1.2 (EN/CHIP_PU)
- net at R14.1: now also U1.4 (GPIO5/ADC2_CH0)
- net at JP2.1 (A): now also U1.8 (GPIO9)
- new net: R7.2, U1.16 (GPIO2/ADC1_CH2)
- new net: R6.2, U1.7 (GPIO8)
- no-connect marks 15 -> 7
Other:
- note removed: "BOOT"
- moved on the sheet: D3, JP2, R14, R3, R6, R7
